File: u4xVCA_v3.sch (EAGLE design)
At the start: 155 parts, among them IC1 OPA1654, IC10 OPA1654, IC2 LM358PW, IC3 V2164SZ, IC4 OPA1654, IC5 OPA1654, IC6 LM358PW, IC7 V2164SZ, IC8 LM4040C25, IC9 LM4040C10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

Commit message: u4xVCA_v3 files
Other:
- note added: "Codex-Modulex"
- note added: "Original design by: Olivier Gillet of Mutable Instruments"
- note added: "info@codex-modulex.com"
- note removed: "Olivier Gillet"
- note removed: "ol.gillet@gmail.com"
Changed lines of the file:
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@@
 <plain>
 <text x="162.56" y="20.32" size="2.54" layer="94">cc-by-sa</text>
-<text x="162.56" y="15.24" size="2.54" layer="94">Olivier Gillet</text>
-<text x="162.56" y="10.16" size="2.54" layer="94">ol.gillet@gmail.com</text>
+<text x="162.56" y="16.002" size="2.54" layer="94">Codex-Modulex</text>
+<text x="162.56" y="11.684" size="2.54" layer="94">info@codex-modulex.com</text>
 <text x="215.9" y="20.32" size="2.54" layer="94">Channel 1</text>
+<text x="162.56" y="5.08" size="1.778" layer="94">Original design by:
+Olivier Gillet of Mutable Instruments</text>
 </plain>
 <instances>
@@
 <plain>
 <text x="162.56" y="20.32" size="2.54" layer="94">cc-by-sa</text>
-<text x="162.56" y="15.24" size="2.54" layer="94">Olivier Gillet</text>
-<text x="162.56" y="10.16" size="2.54" layer="94">ol.gillet@gmail.com</text>
+<text x="162.56" y="16.256" size="2.54" layer="94">Codex-Modulex</text>
+<text x="162.56" y="11.938" size="2.54" layer="94">info@codex-modulex.com</text>
 <text x="215.9" y="20.32" size="2.54" layer="94">Channel 2</text>
+<text x="162.56" y="5.08" size="1.778" layer="94">Original design by:
+Olivier Gillet of Mutable Instruments</text>
 </plain>
 <instances>
@@
 <plain>
 <text x="162.56" y="20.32" size="2.54" layer="94">cc-by-sa</text>
-<text x="162.56" y="15.24" size="2.54" layer="94">Olivier Gillet</text>
-<text x="162.56" y="10.16" size="2.54" layer="94">ol.gillet@gmail.com</text>
+<text x="162.56" y="16.002" size="2.54" layer="94">Codex-Modulex</text>
+<text x="162.56" y="11.938" size="2.54" layer="94">info@codex-modulex.com</text>
 <text x="215.9" y="20.32" size="2.54" layer="94">Channel 3</text>
+<text x="162.56" y="5.08" size="1.778" layer="94">Original design by:
+Olivier Gillet of Mutable Instruments</text>
 </plain>
 <instances>
@@
 <plain>
 <text x="162.56" y="20.32" size="2.54" layer="94">cc-by-sa</text>
-<text x="162.56" y="15.24" size="2.54" layer="94">Olivier Gillet</text>
-<text x="162.56" y="10.16" size="2.54" layer="94">ol.gillet@gmail.com</text>
+<text x="162.56" y="15.748" size="2.54" layer="94">Codex-Modulex</text>
+<text x="162.306" y="11.176" size="2.54" layer="94">info@codex-modulex.com</text>
 <text x="215.9" y="20.32" size="2.54" layer="94">Channel 4</text>
+<text x="162.56" y="5.08" size="1.778" layer="94">Original design by:
+Olivier Gillet of Mutable Instruments</text>
 </plain>
 <instances>
@@
 <plain>
 <text x="195.58" y="83.82" size="2.54" layer="94">cc-by-sa</text>
-<text x="195.58" y="78.74" size="2.54" layer="94">Olivier Gillet</text>
-<text x="195.58" y="73.66" size="2.54" layer="94">ol.gillet@gmail.com</text>
+<text x="195.58" y="79.248" size="2.54" layer="94">Codex-Modulex</text>
+<text x="195.58" y="74.93" size="2.54" layer="94">info@codex-modulex.com</text>
 <text x="248.92" y="83.82" size="2.54" layer="94">Power supply</text>
 <text x="261.62" y="203.2" size="1.778" layer="97">0.41mA delivered</text>
@@
 <text x="261.62" y="200.66" size="1.778" layer="97">0.20mA needed</text>
 <text x="215.9" y="200.66" size="1.778" layer="97">0.32mA needed</text>
+<text x="195.58" y="68.58" size="1.778" layer="94">Original design by:
+Olivier Gillet of Mutable Instruments</text>
 </plain>
 <instances>
@@
 </drawing>
 <compatibility>
+<note version="6.3" minversion="6.2.2" severity="warning">
+Since Version 6.2.2 text objects can contain more than one line,
+which will not be processed correctly with this version.
+</note>
 <note version="8.2" severity="warning">
 Since Version 8.2, EAGLE supports online libraries. The ids
